File: DMG-A20-01.kicad_sch (KiCad schematic)
At the start: 21 parts, among them J1 Cart_Edge_Connector, X1 Unpopulated

Commit message: Add files via upload
Parts:
- X1: value Unpopulated -> 2 MiHz
Connections:
- net P10.R6 renamed ~{RESET}.Out
Other:
- note added: "High = internal. Low = external"
Changed lines of the file:
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@@
+		)
+	)
+	(text "High = internal. \nLow = external"
+		(exclude_from_sim no)
+		(at 152.654 129.286 0)
+		(effects
+			(font
+				(size 1.27 1.27)
+			)
 		)
 	)
@@
 		)
 	)
+	(label "~{RESET}.Out"
+		(at 265.43 116.84 0)
+		(fields_autoplaced yes)
+		(effects
+			(font
+				(size 1.27 1.27)
+			)
+			(justify left bottom)
+		)
+	)
 	(label "A14.Out"
 		(at 31.75 40.64 180)
@@
 		)
 	)
-	(label "P10.R6"
-		(at 72.39 78.74 90)
-		(fields_autoplaced yes)
-		(effects
-			(font
-				(size 1.27 1.27)
-			)
-			(justify left bottom)
-		)
-	)
 	(label "GND"
 		(at 140.97 45.72 270)
@@
 		)
 	)
-	(label "P10.R6"
-		(at 265.43 116.84 0)
-		(fields_autoplaced yes)
-		(effects
-			(font
-				(size 1.27 1.27)
-			)
-			(justify left bottom)
-		)
-	)
 	(label "A7.Out"
 		(at 31.75 68.58 180)
@@
 	(label "D6"
 		(at 49.53 50.8 0)
+		(fields_autoplaced yes)
+		(effects
+			(font
+				(size 1.27 1.27)
+			)
+			(justify left bottom)
+		)
+	)
+	(label "~{RESET}.Out"
+		(at 72.39 78.74 90)
 		(fields_autoplaced yes)
 		(effects
@@
 			)
 		)
-		(property "Value" "Unpopulated"
+		(property "Value" "2 MiHz"
 			(at 173.99 149.8599 90)
 			(effects
